File: hardware/board/harp.device.valve-controller/valve_control.kicad_sch (KiCad schematic)
At the start: 72 parts, among them J1 Screw_Terminal_01x02, J10 Screw_Terminal_01x02, J11 Screw_Terminal_01x02, J12 Screw_Terminal_01x02, J13 Screw_Terminal_01x02, J14 Screw_Terminal_01x02, J15 Screw_Terminal_01x02, J16 Screw_Terminal_01x02, J17 Screw_Terminal_01x02, J18 Screw_Terminal_01x02, J19 Screw_Terminal_01x02, J20 Screw_Terminal_01x02, J3 Screw_Terminal_01x02, J6 Screw_Terminal_01x02, J7 Screw_Terminal_01x02, J9 Screw_Terminal_01x02, U1 MIC4127, U10 MIC4127, U11 MIC4127, U12 MIC4127, U13 MIC4127, U14 MIC4127, U6 MIC4127, U8 MIC4127

Commit message: route pcb
Connections:
- net VPP: no longer C20.2, C21.2, C22.2, C23.2, C24.2, C25.2, C26.2, C29.2, U1.6 (V+), U10.6 (V+), U11.6 (V+), U12.6 (V+), U13.6 (V+), U14.6 (V+), U6.6 (V+), U8.6 (V+)
- new net +5V: C20.2, C21.2, C22.2, C23.2, C24.2, C25.2, C26.2, C29.2, U1.6 (V+), U10.6 (V+), U11.6 (V+), U12.6 (V+), U13.6 (V+), U14.6 (V+), U6.6 (V+), U8.6 (V+)
