File: hardware/board/harp.device.valve-controller/valve_control.kicad_sch (KiCad schematic)
At the start: 52 parts, among them J1 Screw_Terminal_01x02, J10 Screw_Terminal_01x02, J11 Screw_Terminal_01x02, J14 Screw_Terminal_01x02, J3 Screw_Terminal_01x02, J6 Screw_Terminal_01x02, J7 Screw_Terminal_01x02, J9 Screw_Terminal_01x02, Q1 CSD17570Q5B, Q10 CSD17570Q5B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

Commit message: update bom
Parts:
- J1, J10, J11, J14, J3, J6, J7, J9: Manufacturer (none) -> Phoenix Contact; Manufacturer Number (none) -> 1844210; Notes (none) -> mates with Phoenix Contact 1840366
Other:
- note added: "Mates with Phoenix Contact 1840366"

Commit message: prep hw initial release
Parts:
- C20, C21, C22, C23: Link https://www.digikey.com/en/products/detail/walsin-technolog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 -> https://www.digikey.com/en/products/detail/murata-electroni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; Manufacturer Walson Technology Corporation -> Murata Electronics; Manufacturer Number 0402B104K160CT -> GRM155R71H104KE14D; Rated Voltage 16V -> 50V
- Q1, Q10, Q3, Q4, Q5, Q6, Q7, Q8: Link (none) -> https://www.digikey.com/en/products/detail/texas-instrument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; Manufacturer (none) -> Texas Instruments; Manufacturer Number (none) -> CSD17570Q5B
- R14, R17, R18, R21, R22, R24, R25, R8: Link (none) -> https://www.digikey.com/en/products/detail/vishay-dale/RCA0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; Manufacturer (none) -> Vishay Dale; Manufacturer Number (none) -> RCA060310R0FKEAHP; Notes (none) -> 1/3W; Tolerance (none) -> 1%
- U1, U10, U6, U8: Manufacturer (none) -> Microchip Technology
