File: hardware/board/harp.device.valve-controller/isolated_usb_rp2040.kicad_sch (KiCad schematic)
At the start: 50 parts, among them J2 Conn_01x03_Male, J21 Conn_01x03_Male, J4 AudioJack3, J5 USB_C_Receptacle_USB2.0, U2 TPD2EUSB30, U3 ADUM4160, U4 RP2040, U5 W25Q16JVUXIQ, X1 ECS-TXO-2016

Commit message: disambiguate LEDs in schematic
Parts:
- D1, D2: value LED -> LED_GREEN
Changed lines of the file:
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@@
 			)
 		)
-		(property "Value" "LED"
+		(property "Value" "LED_GREEN"
 			(at 265.43 82.55 0)
 			(effects
@@
 			)
 		)
-		(property "Value" "LED"
+		(property "Value" "LED_GREEN"
 			(at 265.43 80.645 0)
 			(effects
