File: hardware/board/harp.device.valve-controller/board_power.kicad_sch (KiCad schematic)
At the start: 26 parts, among them J8 Screw_Terminal_01x02, Q18 SUD19P06-60L-E3, Q2 GSFD4005, U15 LMR51430, U7 rt6150b-33gqw

Commit message: update MPN
Parts:
- U9: Link https://www.digikey.com/en/products/detail/rochester-electr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 -> https://www.digikey.com/en/products/detail/analog-devices-i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; Manufacturer Number MAX5902ACEUT -> MAX5902ACEUT+T
Changed lines of the file:
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@@
 			)
 		)
-		(property "Manufacturer Number" "MAX5902ACEUT"
+		(property "Manufacturer Number" "MAX5902ACEUT+T"
 			(at 92.71 71.12 0)
 			(effects
@@
 			)
 		)
-		(property "Link" "https://www.digikey.com/en/products/detail/rochester-electronics-llc/MAX5902ACEUT/12115092"
+		(property "Link" "https://www.digikey.com/en/products/detail/analog-devices-inc-maxim-integrated/MAX5902ACEUT-T/1781252"
 			(at 92.71 71.12 0)
 			(effects
