File: hardware/board/harp.breakout.mini-clamp/harp.breakout.mini-clamp.kicad_sch (KiCad schematic)
At the start: 9 parts, among them J1 Conn_01x12_Socket, J5 Conn_02x10_Odd_Even, J6 Conn_01x12_Socket, U5 TXB0108

Commit message: route breakout board layout partially
Parts:
- J5: footprint Connector_PinHeader_2.54mm:PinHeader_2x10_P2.54mm_Vertical -> Connector_PinSocket_2.54mm:PinSocket_2x10_P2.54mm_Vertical
Changed lines of the file:
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@@
 			)
 		)
-		(property "Footprint" "Connector_PinHeader_2.54mm:PinHeader_2x10_P2.54mm_Vertical"
+		(property "Footprint" "Connector_PinSocket_2.54mm:PinSocket_2x10_P2.54mm_Vertical"
 			(at 71.12 90.17 0)
 			(effects

Commit message: update breakout
Parts:
- added C5: 1uF, Capacitor_SMD:C_0402_1005Metric_Pad0.74x0.62mm_HandSolder, symbol Device:C
- C1, C2, C3, C4: footprint Capacitor_SMD:C_0402_1005Metric -> Capacitor_SMD:C_0402_1005Metric_Pad0.74x0.62mm_HandSolder
- R1: footprint Resistor_SMD:R_0402_1005Metric -> Resistor_SMD:R_0402_1005Metric_Pad0.72x0.64mm_HandSolder
Connections:
- net +3.3V: now also J5.19 (Pin_19), R1.2, U5.5 (VCCA); no longer J5.1 (Pin_1)
- net +5V: now also J5.17 (Pin_17); no longer J5.3 (Pin_3), R1.2
- net GND: now also C5.2; no longer R1.1
- net IN0: now also J5.1 (Pin_1), U5.10 (A8); no longer J5.19 (Pin_19), U5.1 (A1)
- net IN0_5V: now also J1.10 (Pin_10), U5.11 (B8); no longer J6.1 (Pin_1), U5.20 (B1)
- net IN1: now also J5.3 (Pin_3), U5.9 (A7); no longer J5.17 (Pin_17), U5.2 (A2)
- net IN1_5V: now also J1.7 (Pin_7), U5.12 (B7); no longer J6.4 (Pin_4), U5.19 (B2)
- net IN2: now also J5.5 (Pin_5), U5.8 (A6); no longer J5.15 (Pin_15), U5.3 (A3)
- net IN2_5V: now also J1.4 (Pin_4), U5.13 (B6); no longer J6.7 (Pin_7), U5.18 (B3)
- net IN3: now also J5.7 (Pin_7), U5.7 (A5); no longer J5.13 (Pin_13), U5.4 (A4)
- net IN3_5V: now also J1.1 (Pin_1), U5.14 (B5); no longer J6.10 (Pin_10), U5.17 (B4)
- net OUT0: now also J5.9 (Pin_9), U5.4 (A4); no longer J5.11 (Pin_11), U5.7 (A5)
- net OUT0_5V: now also J6.10 (Pin_10), U5.17 (B4); no longer J1.1 (Pin_1), U5.14 (B5)
- net OUT1: now also J5.11 (Pin_11), U5.3 (A3); no longer J5.9 (Pin_9), U5.8 (A6)
- net OUT1_5V: now also J6.7 (Pin_7), U5.18 (B3); no longer J1.4 (Pin_4), U5.13 (B6)
- net OUT2: now also J5.13 (Pin_13), U5.2 (A2); no longer J5.7 (Pin_7), U5.9 (A7)
- net OUT2_5V: now also J6.4 (Pin_4), U5.19 (B2); no longer J1.7 (Pin_7), U5.12 (B7)
- net OUT3: now also J5.15 (Pin_15), U5.1 (A1); no longer J5.5 (Pin_5), U5.10 (A8)
- net OUT3_5V: now also J6.1 (Pin_1), U5.20 (B1); no longer J1.10 (Pin_10), U5.11 (B8)
- net +3V3: no longer names the net of U5.6 (OE)
- net +3V3: now also R1.1, C5.1; no longer U5.5 (VCCA)
Other:
- note added: "Low pass filter to assert OE after VCC_{A} is stable."
- moved on the sheet: R1

Commit message: update mini clamp breakout bom
Parts:
- J1, J6: Link (none) -> https://www.digikey.com/en/products/detail/3m/37212-62M3-00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; Manufacturer (none) -> 3M; Manufacturer Number (none) -> 37212-62M3-003PL
Changed lines of the file:
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@@
 			)
 		)
-		(property "Datasheet" "~"
+		(property "Datasheet" "https://multimedia.3m.com/mws/media/277250O/3m-shrunk-delta-ribbon-sdr-cable-assembly-ts2120.pdf"
 			(at 231.14 67.31 0)
 			(effects
@@
 		)
 		(property "Description" "Generic connector, single row, 01x12, script generated"
+			(at 231.14 67.31 0)
+			(effects
+				(font
+					(size 1.27 1.27)
+				)
+				(hide yes)
+			)
+		)
+		(property "Link" "https://www.digikey.com/en/products/detail/3m/37212-62M3-003PL/1632992"
+			(at 231.14 67.31 0)
+			(effects
+				(font
+					(size 1.27 1.27)
+				)
+				(hide yes)
+			)
+		)
+		(property "Manufacturer" "3M"
+			(at 231.14 67.31 0)
+			(effects
+				(font
+					(size 1.27 1.27)
+				)
+				(hide yes)
+			)
+		)
+		(property "Manufacturer Number" "37212-62M3-003PL"
 			(at 231.14 67.31 0)
 			(effects
@@
 			)
 		)
-		(property "Datasheet" "~"
+		(property "Datasheet" "https://multimedia.3m.com/mws/media/277250O/3m-shrunk-delta-ribbon-sdr-cable-assembly-ts2120.pdf"
 			(at 231.14 104.14 0)
 			(effects
@@
 		)
 		(property "Description" "Generic connector, single row, 01x12, script generated"
+			(at 231.14 104.14 0)
+			(effects
+				(font
+					(size 1.27 1.27)
+				)
+				(hide yes)
+			)
+		)
+		(property "Link" "https://www.digikey.com/en/products/detail/3m/37212-62M3-003PL/1632992"
+			(at 231.14 104.14 0)
+			(effects
+				(font
+					(size 1.27 1.27)
+				)
+				(hide yes)
+			)
+		)
+		(property "Manufacturer" "3M"
+			(at 231.14 104.14 0)
+			(effects
+				(font
+					(size 1.27 1.27)
+				)
+				(hide yes)
+			)
+		)
+		(property "Manufacturer Number" "37212-62M3-003PL"
 			(at 231.14 104.14 0)
 			(effects
@@
 			)
 		)
-		(property "Datasheet" "~"
+		(property "Datasheet" "https://mm.digikey.com/Volume0/opasdata/d220001/medias/docus/937/Female_Headers.100_DS.pdf"
 			(at 71.12 90.17 0)
 			(effects
